File: electronics/mainboard/mainboard.kicad_sch (KiCad schematic)
At the start: 24 parts, among them Q1 TSM250N02CX_RFG, Q2 TSM250N02CX_RFG, SW1 SW_Push, SW10 SW_Push, SW11 SW_Push, SW12 SW_Push, SW13 SW_Push, SW14 SW_Push, SW15 SW_Push, SW2 SW_Push, SW3 SW_Push, SW4 SW_Push, SW5 SW_Push, SW6 SW_Push, SW7 SW_Push, SW8 SW_Push, SW9 SW_Push, U1 1022

Commit message: modify page layout with version data
Other:
- title: (none) -> Mainboard
Changed lines of the file:
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@@
 (kicad_sch (version 20211123) (generator eeschema)
   (paper "A4")
+  (title_block
+    (title "Mainboard")
+  )
   (junction (at 76.2 48.26) (diameter 0) (color 0 0 0 0)
   )
